File: pcb/large-bridge.kicad_sch (KiCad schematic)
At the start: 0 parts

Commit message: Save progress
Parts:
- added C2: 10u, Capacitor_SMD:C_0603_1608Metric, symbol Device:C
- added R28, R30: 22R, Resistor_SMD:R_0603_1608Metric, symbol Device:R
- added R31: 15k, Resistor_SMD:R_0402_1005Metric, symbol Device:R
- added R36: 2k, Resistor_SMD:R_0402_1005Metric, symbol Device:R
- added U4, U5: TPHR8504PL, Package_DFN_QFN:PQFN-8-EP_6x5mm_P1.27mm_Generic, symbol User_Symbols:TPHR8504PL
Connections:
- new net: R28.2, U5.4 (G)
- new net: R30.2, U4.4 (G)
- new net BST: C2.1
- new net GND: R36.2
- new net HI: R28.1
- new net LO: R30.1
- new net LOW: U4.1 (S), U4.2 (S), U4.3 (S)
- new net OUT: C2.2, R31.1, U4.5 (D), U4.6 (D), U4.7 (D), U4.8 (D), U5.1 (S), U5.2 (S), U5.3 (S)
- new net SNS: R31.2, R36.1
- new net VDD: U5.5 (D), U5.6 (D), U5.7 (D), U5.8 (D)
Other:
- note removed: "TPHR8504PL,LQ(M1W"

Commit message: Save test layout
Parts:
- renumbered C2 to C49, R28 to R34, R30 to R35, R31 to R36, R36 to R37, U4 to U10, U5 to U9
Connections:
- net OUT: no longer U10.6 (D), U10.7 (D), U10.8 (D)
- net VDD: no longer U9.6 (D), U9.7 (D), U9.8 (D)
Changed lines of the file:
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@@
 		(on_board yes)
 		(dnp no)
-		(property "Reference" "U5"
+		(property "Reference" "U9"
 			(at 70.612 52.578 0)
 			(effects
@@
 			)
 		)
-		(pin "7"
-		)
-		(pin "6"
-		)
-		(pin "8"
-		)
 		(pin "5"
 		)
@@
 			(project "combat-control"
 				(path "/38b0a34b-2047-47f6-90d7-ccdf77e8e212/08de4c32-29d6-480e-9b72-c141cc8253af/61412924-99e8-4d1d-998c-c58d470aca1e"
-					(reference "U3")
-					(unit 1)
-				)
-				(path "/38b0a34b-2047-47f6-90d7-ccdf77e8e212/08de4c32-29d6-480e-9b72-c141cc8253af/bae32963-5787-4143-9f83-b032f5349cab"
-					(reference "U6")
-					(unit 1)
-				)
-				(path "/38b0a34b-2047-47f6-90d7-ccdf77e8e212/08de4c32-29d6-480e-9b72-c141cc8253af/e2dc77f2-1da3-4558-9548-0368b6f1c39f"
-					(reference "U5")
+					(reference "U9")
+					(unit 1)
+				)
+				(path "/38b0a34b-2047-47f6-90d7-ccdf77e8e212/08de4c32-29d6-480e-9b72-c141cc8253af/bae32963-5787-4143-9f83-b032f5349cab"
+					(reference "U11")
+					(unit 1)
+				)
+				(path "/38b0a34b-2047-47f6-90d7-ccdf77e8e212/08de4c32-29d6-480e-9b72-c141cc8253af/e2dc77f2-1da3-4558-9548-0368b6f1c39f"
+					(reference "U7")
 					(unit 1)
 				)
@@
 	)
 	(symbol
+		(lib_name "TPHR8504PL_1")
 		(lib_id "User_Symbols:TPHR8504PL")
 		(at 76.2 71.12 0)
@@
 		(on_board yes)
 		(dnp no)
-		(property "Reference" "U4"
+		(property "Reference" "U10"
 			(at 70.612 67.818 0)
 			(effects
@@
 			)
 		)
-		(pin "7"
-		)
-		(pin "6"
-		)
-		(pin "8"
-		)
 		(pin "5"
 		)
@@
 			(project "combat-control"
 				(path "/38b0a34b-2047-47f6-90d7-ccdf77e8e212/08de4c32-29d6-480e-9b72-c141cc8253af/61412924-99e8-4d1d-998c-c58d470aca1e"
-					(reference "U4")
-					(unit 1)
-				)
-				(path "/38b0a34b-2047-47f6-90d7-ccdf77e8e212/08de4c32-29d6-480e-9b72-c141cc8253af/bae32963-5787-4143-9f83-b032f5349cab"
-					(reference "U7")
+					(reference "U10")
+					(unit 1)
+				)
+				(path "/38b0a34b-2047-47f6-90d7-ccdf77e8e212/08de4c32-29d6-480e-9b72-c141cc8253af/bae32963-5787-4143-9f83-b032f5349cab"
+					(reference "U12")
+					(unit 1)
+				)
+				(path "/38b0a34b-2047-47f6-90d7-ccdf77e8e212/08de4c32-29d6-480e-9b72-c141cc8253af/e2dc77f2-1da3-4558-9548-0368b6f1c39f"
+					(reference "U8")
 					(unit 1)
 				)
@@
 		(dnp no)
 		(fields_autoplaced yes)
-		(property "Reference" "C2"
+		(property "Reference" "C49"
 			(at 87.63 55.8799 0)
 			(effects
@@
 			(project ""
 				(path "/38b0a34b-2047-47f6-90d7-ccdf77e8e212/08de4c32-29d6-480e-9b72-c141cc8253af/61412924-99e8-4d1d-998c-c58d470aca1e"
-					(reference "C2")
-					(unit 1)
-				)
-				(path "/38b0a34b-2047-47f6-90d7-ccdf77e8e212/08de4c32-29d6-480e-9b72-c141cc8253af/bae32963-5787-4143-9f83-b032f5349cab"
-					(reference "C3")
-					(unit 1)
-				)
-				(path "/38b0a34b-2047-47f6-90d7-ccdf77e8e212/08de4c32-29d6-480e-9b72-c141cc8253af/e2dc77f2-1da3-4558-9548-0368b6f1c39f"
-					(reference "C1")
+					(reference "C49")
+					(unit 1)
+				)
+				(path "/38b0a34b-2047-47f6-90d7-ccdf77e8e212/08de4c32-29d6-480e-9b72-c141cc8253af/bae32963-5787-4143-9f83-b032f5349cab"
+					(reference "C50")
+					(unit 1)
+				)
+				(path "/38b0a34b-2047-47f6-90d7-ccdf77e8e212/08de4c32-29d6-480e-9b72-c141cc8253af/e2dc77f2-1da3-4558-9548-0368b6f1c39f"
+					(reference "C48")
 					(unit 1)
 				)
@@
 		(dnp no)
 		(fields_autoplaced yes)
-		(property "Reference" "R28"
+		(property "Reference" "R34"
 			(at 62.23 49.53 90)
 			(effects
@@
 			(project "combat-control"
 				(path "/38b0a34b-2047-47f6-90d7-ccdf77e8e212/08de4c32-29d6-480e-9b72-c141cc8253af/61412924-99e8-4d1d-998c-c58d470aca1e"
-					(reference "R28")
-					(unit 1)
-				)
-				(path "/38b0a34b-2047-47f6-90d7-ccdf77e8e212/08de4c32-29d6-480e-9b72-c141cc8253af/bae32963-5787-4143-9f83-b032f5349cab"
 					(reference "R34")
+					(unit 1)
+				)
+				(path "/38b0a34b-2047-47f6-90d7-ccdf77e8e212/08de4c32-29d6-480e-9b72-c141cc8253af/bae32963-5787-4143-9f83-b032f5349cab"
+					(reference "R38")
+					(unit 1)
+				)
+				(path "/38b0a34b-2047-47f6-90d7-ccdf77e8e212/08de4c32-29d6-480e-9b72-c141cc8253af/e2dc77f2-1da3-4558-9548-0368b6f1c39f"
+					(reference "R30")
 					(unit 1)
 				)
@@
 		(dnp no)
 		(fields_autoplaced yes)
-		(property "Reference" "R31"
+		(property "Reference" "R36"
 			(at 86.36 68.5799 0)
 			(effects
@@
 			(project "combat-control"
 				(path "/38b0a34b-2047-47f6-90d7-ccdf77e8e212/08de4c32-29d6-480e-9b72-c141cc8253af/61412924-99e8-4d1d-998c-c58d470aca1e"
-					(reference "R31")
-					(unit 1)
-				)
-				(path "/38b0a34b-2047-47f6-90d7-ccdf77e8e212/08de4c32-29d6-480e-9b72-c141cc8253af/bae32963-5787-4143-9f83-b032f5349cab"
-					(reference "R37")
+					(reference "R36")
+					(unit 1)
+				)
+				(path "/38b0a34b-2047-47f6-90d7-ccdf77e8e212/08de4c32-29d6-480e-9b72-c141cc8253af/bae32963-5787-4143-9f83-b032f5349cab"
+					(reference "R40")
+					(unit 1)
+				)
+				(path "/38b0a34b-2047-47f6-90d7-ccdf77e8e212/08de4c32-29d6-480e-9b72-c141cc8253af/e2dc77f2-1da3-4558-9548-0368b6f1c39f"
+					(reference "R32")
 					(unit 1)
 				)
@@
 		(dnp no)
 		(fields_autoplaced yes)
-		(property "Reference" "#PWR016"
+		(property "Reference" "#PWR078"
 			(at 83.82 95.25 0)
 			(effects
@@
 			(project "combat-control"
 				(path "/38b0a34b-2047-47f6-90d7-ccdf77e8e212/08de4c32-29d6-480e-9b72-c141cc8253af/61412924-99e8-4d1d-998c-c58d470aca1e"
-					(reference "#PWR016")
-					(unit 1)
-				)
-				(path "/38b0a34b-2047-47f6-90d7-ccdf77e8e212/08de4c32-29d6-480e-9b72-c141cc8253af/bae32963-5787-4143-9f83-b032f5349cab"
-					(reference "#PWR020")
+					(reference "#PWR078")
+					(unit 1)
+				)
+				(path "/38b0a34b-2047-47f6-90d7-ccdf77e8e212/08de4c32-29d6-480e-9b72-c141cc8253af/bae32963-5787-4143-9f83-b032f5349cab"
+					(reference "#PWR080")
+					(unit 1)
+				)
+				(path "/38b0a34b-2047-47f6-90d7-ccdf77e8e212/08de4c32-29d6-480e-9b72-c141cc8253af/e2dc77f2-1da3-4558-9548-0368b6f1c39f"
+					(reference "#PWR076")
 					(unit 1)
 				)
@@
 		(dnp no)
 		(fields_autoplaced yes)
-		(property "Reference" "R30"
+		(property "Reference" "R35"
 			(at 62.23 64.77 90)
 			(effects
@@
 			(project "combat-control"
 				(path "/38b0a34b-2047-47f6-90d7-ccdf77e8e212/08de4c32-29d6-480e-9b72-c141cc8253af/61412924-99e8-4d1d-998c-c58d470aca1e"
-					(reference "R29")
-					(unit 1)
-				)
-				(path "/38b0a34b-2047-47f6-90d7-ccdf77e8e212/08de4c32-29d6-480e-9b72-c141cc8253af/bae32963-5787-4143-9f83-b032f5349cab"
 					(reference "R35")
 					(unit 1)
 				)
-				(path "/38b0a34b-2047-47f6-90d7-ccdf77e8e212/08de4c32-29d6-480e-9b72-c141cc8253af/e2dc77f2-1da3-4558-9548-0368b6f1c39f"
-					(reference "R30")
+				(path "/38b0a34b-2047-47f6-90d7-ccdf77e8e212/08de4c32-29d6-480e-9b72-c141cc8253af/bae32963-5787-4143-9f83-b032f5349cab"
+					(reference "R39")
+					(unit 1)
+				)
+				(path "/38b0a34b-2047-47f6-90d7-ccdf77e8e212/08de4c32-29d6-480e-9b72-c141cc8253af/e2dc77f2-1da3-4558-9548-0368b6f1c39f"
+					(reference "R31")
 					(unit 1)
 				)
@@
 		(dnp no)
 		(fields_autoplaced yes)
-		(property "Reference" "#PWR015"
+		(property "Reference" "#PWR077"
 			(at 76.2 52.07 0)
 			(effects
@@
 			(project "combat-control"
 				(path "/38b0a34b-2047-47f6-90d7-ccdf77e8e212/08de4c32-29d6-480e-9b72-c141cc8253af/61412924-99e8-4d1d-998c-c58d470aca1e"
-					(reference "#PWR015")
-					(unit 1)
-				)
-				(path "/38b0a34b-2047-47f6-90d7-ccdf77e8e212/08de4c32-29d6-480e-9b72-c141cc8253af/bae32963-5787-4143-9f83-b032f5349cab"
-					(reference "#PWR019")
+					(reference "#PWR077")
+					(unit 1)
+				)
+				(path "/38b0a34b-2047-47f6-90d7-ccdf77e8e212/08de4c32-29d6-480e-9b72-c141cc8253af/bae32963-5787-4143-9f83-b032f5349cab"
+					(reference "#PWR079")
+					(unit 1)
+				)
+				(path "/38b0a34b-2047-47f6-90d7-ccdf77e8e212/08de4c32-29d6-480e-9b72-c141cc8253af/e2dc77f2-1da3-4558-9548-0368b6f1c39f"
+					(reference "#PWR075")
 					(unit 1)
 				)
@@
 		(dnp no)
 		(fields_autoplaced yes)
-		(property "Reference" "R36"
+		(property "Reference" "R37"
 			(at 86.36 81.2799 0)
 			(effects
@@
 			(project "combat-control"
 				(path "/38b0a34b-2047-47f6-90d7-ccdf77e8e212/08de4c32-29d6-480e-9b72-c141cc8253af/61412924-99e8-4d1d-998c-c58d470aca1e"
-					(reference "R32")
-					(unit 1)
-				)
-				(path "/38b0a34b-2047-47f6-90d7-ccdf77e8e212/08de4c32-29d6-480e-9b72-c141cc8253af/bae32963-5787-4143-9f83-b032f5349cab"
-					(reference "R38")
-					(unit 1)
-				)
-				(path "/38b0a34b-2047-47f6-90d7-ccdf77e8e212/08de4c32-29d6-480e-9b72-c141cc8253af/e2dc77f2-1da3-4558-9548-0368b6f1c39f"
-					(reference "R36")
-					(unit 1)
-				)
+					(reference "R37")
+					(unit 1)
+				)
+				(path "/38b0a34b-2047-47f6-90d7-ccdf77e8e212/08de4c32-29d6-480e-9b72-c141cc8253af/bae32963-5787-4143-9f83-b032f5349cab"
+					(reference "R41")
+					(unit 1)
+				)
+				(path "/38b0a34b-2047-47f6-90d7-ccdf77e8e212/08de4c32-29d6-480e-9b72-c141cc8253af/e2dc77f2-1da3-4558-9548-0368b6f1c39f"
+					(reference "R33")
+					(unit 1)
+				)
