File: pcb/combat-control.kicad_sch (KiCad schematic)
At the start: 0 parts

Commit message: Select parts
Other:
- added sheet LargeMotor (large-motor.kicad_sch)
- added sheet SmallMotor1 (small-motor.kicad_sch)
- added sheet SmallMotor2 (small-motor.kicad_sch)
- note added: "ESP32-S3FH4R2"
Changed lines of the file:
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@@
 	(generator_version "8.0")
 	(paper "A4")
+	(text "ESP32-S3FH4R2"
+		(exclude_from_sim no)
+		(at 50.292 66.802 0)
+		(effects
+			(font
+				(size 1.27 1.27)
+			)
+		)
+	)
+	(sheet
+		(at 148.59 86.36)
+		(size 27.94 15.24)
+		(fields_autoplaced yes)
+		(stroke
+			(width 0.1524)
+			(type solid)
+		)
+		(fill
+			(color 0 0 0 0.0000)
+		)
+		(property "Sheetname" "LargeMotor"
+			(at 148.59 85.6484 0)
+			(effects
+				(font
+					(size 1.27 1.27)
+				)
+				(justify left bottom)
+			)
+		)
+		(property "Sheetfile" "large-motor.kicad_sch"
+			(at 148.59 102.1846 0)
+			(effects
+				(font
+					(size 1.27 1.27)
+				)
+				(justify left top)
+			)
+		)
+		(instances
+			(project "combat-control"
+				(path "/38b0a34b-2047-47f6-90d7-ccdf77e8e212"
+					(page "10")
+				)
+			)
+		)
+	)
+	(sheet
+		(at 80.01 124.46)
+		(size 30.48 15.24)
+		(fields_autoplaced yes)
+		(stroke
+			(width 0.1524)
+			(type solid)
+		)
+		(fill
+			(color 0 0 0 0.0000)
+		)
+		(property "Sheetname" "SmallMotor2"
+			(at 80.01 123.7484 0)
+			(effects
+				(font
+					(size 1.27 1.27)
+				)
+				(justify left bottom)
+			)
+		)
+		(property "Sheetfile" "small-motor.kicad_sch"
+			(at 80.01 140.2846 0)
+			(effects
+				(font
+					(size 1.27 1.27)
+				)
+				(justify left top)
+			)
+		)
+		(instances
+			(project "combat-control"
+				(path "/38b0a34b-2047-47f6-90d7-ccdf77e8e212"
+					(page "6")
+				)
+			)
+		)
+	)
+	(sheet
+		(at 80.01 92.71)
+		(size 30.48 15.24)
+		(fields_autoplaced yes)
+		(stroke
+			(width 0.1524)
+			(type solid)
+		)
+		(fill
+			(color 0 0 0 0.0000)
+		)
+		(property "Sheetname" "SmallMotor1"
+			(at 80.01 91.9984 0)
+			(effects
+				(font
+					(size 1.27 1.27)
+				)
+				(justify left bottom)
+			)
+		)
+		(property "Sheetfile" "small-motor.kicad_sch"
+			(at 80.01 108.5346 0)
+			(effects
+				(font
+					(size 1.27 1.27)
+				)
+				(justify left top)
+			)
+		)
+		(instances
+			(project "combat-control"
+				(path "/38b0a34b-2047-47f6-90d7-ccdf77e8e212"
+					(page "3")
+				)
+			)
+		)
+	)
 	(sheet_instances
 		(path "/"

Commit message: Save progress
Parts:
- added C19: 4u7, Capacitor_SMD:C_0402_1005Metric, symbol Device:C
- added C25, C29, C35, C36, C37: 100n, Capacitor_SMD:C_0402_1005Metric, symbol Device:C
- added C30, C31, C32, C34: 2m2, User_Footprints:C_D10xL16_Horizontal, symbol Device:C
- added C33: 10u, Capacitor_SMD:C_0603_1608Metric, symbol Device:C
- added C38: 10u, Capacitor_SMD:C_0402_1005Metric, symbol Device:C
- added J7, J8: Conn_01x01_Pin, MountingHole:MountingHole_3.2mm_M3_Pad_Via, symbol Connector:Conn_01x01_Pin
- added U10: ESP32-S3, Package_DFN_QFN:QFN-56-1EP_7x7mm_P0.4mm_EP4x4mm, symbol MCU_Espressif:ESP32-S3
- added U11: ICM-42688-P, Package_LGA:LGA-14_3x2.5mm_P0.5mm_LayoutBorder3x4y, symbol User_Symbols:ICM-42688-P
- added U12: LP38690SD, Package_DFN_QFN:DFN-6-1EP_3x3mm_P0.95mm_EP1.7x2.6mm, symbol User_Symbols:LP38690SD-3.3
Connections:
- new net: U10.2 (VDD3P3), U10.3 (VDD3P3)
- new net: U10.55 (VDDA), U10.56 (VDDA)
- new net +3V3: C19.1, C25.1, C29.1, C37.1, C38.1, U11.5 (VDDIO), U11.8 (VDD), U12.4 (OUT), U12.5 (SNS)
- new net +5V: C33.1, C35.1, C36.1, U12.1 (IN), U12.6 (IN)
- new net CLK: U11.13 (CLK)
- new net GCS: U11.12 (CS)
- new net GINT: U11.4 (INT1)
- new net GND: C19.2, C25.2, C29.2, C30.2, C31.2, C32.1, C33.2, C34.2, C35.2, C36.2, C37.2, C38.2, J8.1 (Pin_1), U10.57 (GND), U11.11 (RESV), U11.6 (GND), U11.7 (RESV), U12.2 (GND), U12.7 (PAD)
- new net MISO: U11.1 (SDO)
- new net MOSI: U11.14 (SDI)
- new net VDD: C30.1, C31.1, C32.2, C34.1, J7.1 (Pin_1)
- no-connect marks 0 -> 1
Other:
- sheet LargeMotor ports: added EN, INA, INB, INC, ISNS, SNSA, SNSB, SNSC; removed none
- sheet SmallMotor1 ports: added ILIM, INA, INB, INC, SNSA, SNSB, SNSC; removed none
- sheet SmallMotor2 ports: added ILIM, INA, INB, INC, SNSA, SNSB, SNSC; removed none
- note added: "Battery"
- note added: "Bulk Capacitors"
- note added: "IMU"
- note added: "LGS5145"
- note added: "Low Noise LDO"
- note removed: "ESP32-S3FH4R2"

Commit message: Save test layout
Parts:
- removed C33: 10u, Capacitor_SMD:C_0603_1608Metric, symbol Device:C
- removed C35, C36, C37: 100n, Capacitor_SMD:C_0402_1005Metric, symbol Device:C
- removed C38: 10u, Capacitor_SMD:C_0402_1005Metric, symbol Device:C
- removed U12: LP38690SD, Package_DFN_QFN:DFN-6-1EP_3x3mm_P0.95mm_EP1.7x2.6mm, symbol User_Symbols:LP38690SD-3.3
- added AE1: Antenna_Shield, Connector_Coaxial:U.FL_Molex_MCRF_73412-0110_Vertical, symbol Device:Antenna_Shield
- added C10, C13: C, Resistor_SMD:R_0402_1005Metric, symbol Device:C
- added C11, C18, C8: 1u, Capacitor_SMD:C_0402_1005Metric, symbol Device:C
- added C12: 10n, Capacitor_SMD:C_0402_1005Metric, symbol Device:C
- added C14, C15, C16, C17, C20: 100n, Capacitor_SMD:C_0402_1005Metric, symbol Device:C
- added C19, C21, C22: C, Capacitor_SMD:C_0402_1005Metric, symbol Device:C
- added C9: 10u, Capacitor_SMD:C_0402_1005Metric, symbol Device:C
- added L1, L3, L4: L, Inductor_SMD:L_0402_1005Metric, symbol Device:L
- added L2: 2nH, Inductor_SMD:L_0402_1005Metric, symbol Device:L
- added Y1: 40MHz, Crystal:Crystal_SMD_2520-4Pin_2.5x2.0mm, symbol Device:Crystal_GND24
- renumbered C19 to C1, C25 to C2, C29 to C3, C30 to C4, C32 to C5, C34 to C6, C31 to C7, J7 to J1, J8 to J2, U11 to U1, U10 to U2
Connections:
- net +3V3: now also U2.20 (VDD3P3_RTC), U2.29 (VDD_SPI), U2.4 (CHIP_PU), U2.46 (VDD3P3_CPU), U2.55 (VDDA), U2.56 (VDDA), C11.1, C12.1, C14.1, C16.1, C17.1, C18.1, C20.1, C8.1, C9.1, L2.1
- net GND: now also AE1.2 (Shield), C10.2, C11.2, C12.2, C13.2, C14.2, C15.2, C16.2, C17.2, C18.2, C19.2, C20.2, C21.2, C22.2, C8.2, C9.2, Y1.2, Y1.4
- net at U2.1 (LNA_IN): now also C19.1, L3.1
- net VDD3: now reaches U2.2 (VDD3P3), U2.3 (VDD3P3)
- net VDD3: now also C15.1, L2.2
- net STP: now reaches U2.52 (GPIO46)
- net STP: now also U2.8 (GPIO3)
- net at U2.53 (XTAL_N): now also C13.1, Y1.3
- net at U2.54 (XTAL_P): now also L1.2
- new net: AE1.1 (A), C21.1, L3.2, L4.1
- new net: C10.1, L1.1, Y1.1
- new net: C22.1, L4.2
- no-connect marks 1 -> 11
Other:
- note added: "LMR50410XDBVR"
- note added: "LT8609"
- note added: "Set EFUSE_VDD_SPI_FORCE and EFUSE_VDD_SPI_TIEH"
- note removed: "Low Noise LDO"
- moved on the sheet: U2

Commit message: Save layout
Parts:
- removed C4, C5, C6, C7: 2m2, User_Footprints:C_D10xL16_Horizontal, symbol Device:C
Connections:
- net IFIG: now reaches U2.5 (GPIO0)
- net IFIG: now also U2.51 (GPIO45)
- no-connect marks 11 -> 10
Other:
- note removed: "Bulk Capacitors"
