File: pcb/large-motor.kicad_sch (KiCad schematic)
At the start: 1 part, among them U1 ACS781xLRTR-100B

Commit message: Save progress
Parts:
- added C10, C9: 10u, Capacitor_SMD:C_0805_2012Metric, symbol Device:C
- added C4, C6, C8: 100n, Capacitor_SMD:C_0402_1005Metric, symbol Device:C
- added C5: 470n, Capacitor_SMD:C_0603_1608Metric, symbol Device:C
- added C7: 22u, Capacitor_SMD:C_0805_2012Metric, symbol Device:C
- added R27: 10k, Resistor_SMD:R_0402_1005Metric, symbol Device:R
- added U8: DRV8328B, Package_DFN_QFN:QFN-28-1EP_4x4mm_P0.4mm_EP2.6x2.6mm, symbol User_Symbols:DRV8328B
Connections:
- net +3V3: now reaches U1.1 (VCC)
- net +3V3: now also C4.1, U8.21 (INLC), U8.22 (INLB), U8.23 (INLA), U8.26 (DLVL)
- net GND: now reaches U1.2 (GND)
- net GND: now also U1.6 (IP-), C10.2, C4.2, C6.2, C7.2, C8.2, C9.2, R27.2, U8.17 (LSS), U8.28 (GND), U8.29 (PAD)
- net ISNS: now reaches U1.3 (VOUT)
- net LOW: now reaches U1.5 (IP+)
- new net: R27.1, U8.27 (DT)
- new net: C5.1, U8.2 (CPL)
- new net: C5.2, U8.3 (CPH)
- new net BSTA: U8.5 (BSTA)
- new net BSTB: U8.9 (BSTB)
- new net BSTC: U8.13 (BSTC)
- new net EN: U8.25 (~{SLP})
- new net GVDD: C6.1, C7.1, U8.4 (GVDD)
- new net HIA: U8.7 (GHA)
- new net HIB: U8.11 (GHB)
- new net HIC: U8.15 (GHC)
- new net INA: U8.20 (INHA)
- new net INB: U8.19 (INHB)
- new net INC: U8.18 (INHC)
- new net LOA: U8.8 (GLA)
- new net LOB: U8.12 (GLB)
- new net LOC: U8.16 (GLC)
- new net OUTA: U8.6 (SHA)
- new net OUTB: U8.10 (SHB)
- new net OUTC: U8.14 (SHC)
- new net VDD: C10.1, C8.1, C9.1, U8.1 (PVDD)
- no-connect marks 2 -> 3
Other:
- removed sheet LargeBridgeC
- added sheet LargeBridgeA2 (large-bridge.kicad_sch)
- sheet LargeBridgeA ports: added BST, HI, LO, LOW, OUT, SNS; removed none
- sheet LargeBridgeB ports: added BST, HI, LO, LOW, OUT, SNS; removed none
- note removed: "DRV8328B"
- moved on the sheet: U1

Commit message: Save test layout
Parts:
- renumbered C7 to C41, C6 to C42, C10 to C43, C9 to C44, C5 to C45, C8 to C46, C4 to C47, R27 to R29, U8 to U5, U1 to U6
Changed lines of the file:
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@@
 		(dnp no)
 		(fields_autoplaced yes)
-		(property "Reference" "#PWR031"
+		(property "Reference" "#PWR063"
 			(at 33.02 69.85 0)
 			(effects
@@
 			(project "combat-control"
 				(path "/38b0a34b-2047-47f6-90d7-ccdf77e8e212/08de4c32-29d6-480e-9b72-c141cc8253af"
-					(reference "#PWR031")
+					(reference "#PWR063")
 					(unit 1)
 				)
@@
 		(dnp no)
 		(fields_autoplaced yes)
-		(property "Reference" "#PWR027"
+		(property "Reference" "#PWR074"
 			(at 177.8 67.31 0)
 			(effects
@@
 			(project "combat-control"
 				(path "/38b0a34b-2047-47f6-90d7-ccdf77e8e212/08de4c32-29d6-480e-9b72-c141cc8253af"
-					(reference "#PWR027")
+					(reference "#PWR074")
 					(unit 1)
 				)
@@
 		(dnp no)
 		(fields_autoplaced yes)
-		(property "Reference" "#PWR023"
+		(property "Reference" "#PWR070"
 			(at 154.94 90.17 0)
 			(effects
@@
 			(project "combat-control"
 				(path "/38b0a34b-2047-47f6-90d7-ccdf77e8e212/08de4c32-29d6-480e-9b72-c141cc8253af"
-					(reference "#PWR023")
+					(reference "#PWR070")
 					(unit 1)
 				)
@@
 		(dnp no)
 		(fields_autoplaced yes)
-		(property "Reference" "#PWR032"
+		(property "Reference" "#PWR061"
 			(at 22.86 69.85 0)
 			(effects
@@
 			(project "combat-control"
 				(path "/38b0a34b-2047-47f6-90d7-ccdf77e8e212/08de4c32-29d6-480e-9b72-c141cc8253af"
-					(reference "#PWR032")
+					(reference "#PWR061")
 					(unit 1)
 				)
@@
 		(on_board yes)
 		(dnp no)
-		(property "Reference" "C7"
+		(property "Reference" "C41"
 			(at 25.908 55.88 0)
 			(effects
@@
 			(project "combat-control"
 				(path "/38b0a34b-2047-47f6-90d7-ccdf77e8e212/08de4c32-29d6-480e-9b72-c141cc8253af"
-					(reference "C7")
+					(reference "C41")
 					(unit 1)
 				)
@@
 		(dnp no)
 		(fields_autoplaced yes)
-		(property "Reference" "C6"
+		(property "Reference" "C42"
 			(at 36.83 55.8799 0)
 			(effects
@@
 			(project ""
 				(path "/38b0a34b-2047-47f6-90d7-ccdf77e8e212/08de4c32-29d6-480e-9b72-c141cc8253af"
-					(reference "C6")
+					(reference "C42")
 					(unit 1)
 				)
@@
 		(dnp no)
 		(fields_autoplaced yes)
-		(property "Reference" "#PWR014"
+		(property "Reference" "#PWR064"
 			(at 54.61 68.58 0)
 			(effects
@@
 			(project ""
 				(path "/38b0a34b-2047-47f6-90d7-ccdf77e8e212/08de4c32-29d6-480e-9b72-c141cc8253af"
-					(reference "#PWR014")
+					(reference "#PWR064")
 					(unit 1)
 				)
@@
 		(dnp no)
 		(fields_autoplaced yes)
-		(property "Reference" "#PWR029"
+		(property "Reference" "#PWR069"
 			(at 78.74 97.79 0)
 			(effects
@@
 			(project "combat-control"
 				(path "/38b0a34b-2047-47f6-90d7-ccdf77e8e212/08de4c32-29d6-480e-9b72-c141cc8253af"
-					(reference "#PWR029")
+					(reference "#PWR069")
 					(unit 1)
 				)
@@
 		(dnp no)
 		(fields_autoplaced yes)
-		(property "Reference" "#PWR025"
+		(property "Reference" "#PWR066"
 			(at 53.34 107.95 0)
 			(effects
@@
 			(project "combat-control"
 				(path "/38b0a34b-2047-47f6-90d7-ccdf77e8e212/08de4c32-29d6-480e-9b72-c141cc8253af"
-					(reference "#PWR025")
+					(reference "#PWR066")
 					(unit 1)
 				)
@@
 		(on_board yes)
 		(dnp no)
-		(property "Reference" "C9"
+		(property "Reference" "C44"
 			(at 49.022 38.1 0)
 			(effects
@@
 			(project "combat-control"
 				(path "/38b0a34b-2047-47f6-90d7-ccdf77e8e212/08de4c32-29d6-480e-9b72-c141cc8253af"
-					(reference "C9")
+					(reference "C44")
 					(unit 1)
 				)
@@
 		(dnp no)
 		(fields_autoplaced yes)
-		(property "Reference" "#PWR022"
+		(property "Reference" "#PWR071"
 			(at 167.64 72.39 0)
 			(effects
@@
 			(project ""
 				(path "/38b0a34b-2047-47f6-90d7-ccdf77e8e212/08de4c32-29d6-480e-9b72-c141cc8253af"
-					(reference "#PWR022")
+					(reference "#PWR071")
 					(unit 1)
 				)
@@
 		(dnp no)
 		(fields_autoplaced yes)
-		(property "Reference" "C8"
+		(property "Reference" "C46"
 			(at 59.69 38.0999 0)
 			(effects
@@
 			(project "combat-control"
 				(path "/38b0a34b-2047-47f6-90d7-ccdf77e8e212/08de4c32-29d6-480e-9b72-c141cc8253af"
-					(reference "C8")
+					(reference "C46")
 					(unit 1)
 				)
@@
 		(dnp no)
 		(fields_autoplaced yes)
-		(property "Reference" "R27"
+		(property "Reference" "R29"
 			(at 55.88 93.9799 0)
 			(effects
@@
 			(project ""
 				(path "/38b0a34b-2047-47f6-90d7-ccdf77e8e212/08de4c32-29d6-480e-9b72-c141cc8253af"
-					(reference "R27")
+					(reference "R29")
 					(unit 1)
 				)
@@
 		(dnp no)
 		(fields_autoplaced yes)
-		(property "Reference" "#PWR017"
+		(property "Reference" "#PWR067"
 			(at 66.04 34.29 0)
 			(effects
@@
 			(project ""
 				(path "/38b0a34b-2047-47f6-90d7-ccdf77e8e212/08de4c32-29d6-480e-9b72-c141cc8253af"
-					(reference "#PWR017")
+					(reference "#PWR067")
 					(unit 1)
 				)
@@
 		(on_board yes)
 		(dnp no)
-		(property "Reference" "U1"
+		(property "Reference" "U6"
 			(at 162.306 71.628 0)
 			(effects
@@
 			(project ""
 				(path "/38b0a34b-2047-47f6-90d7-ccdf77e8e212/08de4c32-29d6-480e-9b72-c141cc8253af"
-					(reference "U1")
+					(reference "U6")
 					(unit 1)
 				)
@@
 		(dnp no)
 		(fields_autoplaced yes)
-		(property "Reference" "#PWR021"
+		(property "Reference" "#PWR072"
 			(at 167.64 95.25 0)
 			(effects
@@
 			(project ""
 				(path "/38b0a34b-2047-47f6-90d7-ccdf77e8e212/08de4c32-29d6-480e-9b72-c141cc8253af"
-					(reference "#PWR021")
+					(reference "#PWR072")
 					(unit 1)
 				)
@@
 		(on_board yes)
 		(dnp no)
-		(property "Reference" "C10"
+		(property "Reference" "C43"
 			(at 38.862 38.1 0)
 			(effects
@@
 			(project "combat-control"
 				(path "/38b0a34b-2047-47f6-90d7-ccdf77e8e212/08de4c32-29d6-480e-9b72-c141cc8253af"
-					(reference "C10")
+					(reference "C43")
 					(unit 1)
 				)
@@
 		(dnp no)
 		(fields_autoplaced yes)
-		(property "Reference" "C4"
+		(property "Reference" "C47"
 			(at 181.61 53.3399 0)
 			(effects
@@
 			(project ""
 				(path "/38b0a34b-2047-47f6-90d7-ccdf77e8e212/08de4c32-29d6-480e-9b72-c141cc8253af"
-					(reference "C4")
+					(reference "C47")
 					(unit 1)
 				)
@@
 		(dnp no)
 		(fields_autoplaced yes)
-		(property "Reference" "#PWR028"
+		(property "Reference" "#PWR073"
 			(at 177.8 52.07 0)
 			(effects
@@
 			(project "combat-control"
 				(path "/38b0a34b-2047-47f6-90d7-ccdf77e8e212/08de4c32-29d6-480e-9b72-c141cc8253af"
-					(reference "#PWR028")
+					(reference "#PWR073")
 					(unit 1)
 				)
@@
 		(dnp no)
 		(fields_autoplaced yes)
-		(property "Reference" "#PWR030"
+		(property "Reference" "#PWR065"
 			(at 57.15 86.36 0)
 			(effects
@@
 			(project "combat-control"
 				(path "/38b0a34b-2047-47f6-90d7-ccdf77e8e212/08de4c32-29d6-480e-9b72-c141cc8253af"
-					(reference "#PWR030")
+					(reference "#PWR065")
 					(unit 1)
 				)
@@
 		(dnp no)
 		(fields_autoplaced yes)
-		(property "Reference" "U8"
+		(property "Reference" "U5"
 			(at 68.2341 43.18 0)
 			(effects
@@
 			(project ""
 				(path "/38b0a34b-2047-47f6-90d7-ccdf77e8e212/08de4c32-29d6-480e-9b72-c141cc8253af"
-					(reference "U8")
+					(reference "U5")
 					(unit 1)
 				)
@@
 		(dnp no)
 		(fields_autoplaced yes)
-		(property "Reference" "#PWR033"
+		(property "Reference" "#PWR062"
 			(at 26.67 45.72 0)
 			(effects
@@
 			(project "combat-control"
 				(path "/38b0a34b-2047-47f6-90d7-ccdf77e8e212/08de4c32-29d6-480e-9b72-c141cc8253af"
-					(reference "#PWR033")
+					(reference "#PWR062")
 					(unit 1)
 				)
@@
 		(on_board yes)
 		(dnp no)
-		(property "Reference" "C5"
+		(property "Reference" "C45"
 			(at 46.482 57.658 90)
 			(effects
@@
 			(project ""
 				(path "/38b0a34b-2047-47f6-90d7-ccdf77e8e212/08de4c32-29d6-480e-9b72-c141cc8253af"
-					(reference "C5")
+					(reference "C45")
 					(unit 1)
 				)
@@
 		(dnp no)
 		(fields_autoplaced yes)
-		(property "Reference" "#PWR024"
+		(property "Reference" "#PWR068"
 			(at 66.04 105.41 0)
 			(effects
@@
 			(project ""
 				(path "/38b0a34b-2047-47f6-90d7-ccdf77e8e212/08de4c32-29d6-480e-9b72-c141cc8253af"
-					(reference "#PWR024")
-					(unit 1)
-				)
+					(reference "#PWR068")
+					(unit 1)
+				)

Commit message: Save layout
Parts:
- added C4, C5: 2m2, User_Footprints:C_D10xL16_Horizontal, symbol Device:C
- added J10, J11, J9: Conn_01x01_Pin, MountingHole:MountingHole_3.2mm_M3_Pad_Via, symbol Connector:Conn_01x01_Pin
Connections:
- net GND: now also U6.5 (IP+); no longer U6.6 (IP-)
- net LOW: now also U6.6 (IP-), C4.2, C5.1; no longer U6.5 (IP+)
- net OUTA: now also J9.1 (Pin_1)
- net OUTB: now also J10.1 (Pin_1)
- net OUTC: now also J11.1 (Pin_1)
- net VDD: now also C4.1, C5.2
