File: pcb/small-bridge.kicad_sch (KiCad schematic)
At the start: 6 parts, among them Q1 AON7544, Q2 AON7544

Commit message: Save progress
Parts:
- added C12: 1u, Capacitor_SMD:C_0402_1005Metric, symbol Device:C
- R1: value 10R -> 22R; LCSC C25077 -> C25092
- R20: renamed from R2; value 10R -> 22R; LCSC C25077 -> C25092
- renumbered Q2 to Q10, Q1 to Q9, R3 to R21, R4 to R22
Connections:
- net OUT: now also C12.2
- net CP renamed SNS
- net PL renamed LOW
- new net BST: C12.1
Other:
- moved on the sheet: Q10, Q9, R20, R21, R22

Commit message: Save test layout
Parts:
- renumbered C12 to C31, R1 to R21, R20 to R22, R21 to R23, R22 to R24
Changed lines of the file:
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@@
 		(dnp no)
 		(fields_autoplaced yes)
-		(property "Reference" "#PWR010"
+		(property "Reference" "#PWR057"
 			(at 63.5 52.07 0)
 			(effects
@@
 			(project "combat-control"
 				(path "/38b0a34b-2047-47f6-90d7-ccdf77e8e212/5bc2eb48-ba05-4947-b6cc-1fab53bcabc8/31e52373-a2dc-44cb-afdb-9746210f2a01"
-					(reference "#PWR010")
+					(reference "#PWR057")
 					(unit 1)
 				)
 				(path "/38b0a34b-2047-47f6-90d7-ccdf77e8e212/5bc2eb48-ba05-4947-b6cc-1fab53bcabc8/37cfab98-42f4-441d-a436-14a61a241678"
-					(reference "#PWR05")
+					(reference "#PWR044")
 					(unit 1)
 				)
 				(path "/38b0a34b-2047-47f6-90d7-ccdf77e8e212/5bc2eb48-ba05-4947-b6cc-1fab53bcabc8/f6e61053-1e52-4f8f-88d6-a469198d56c4"
-					(reference "#PWR012")
+					(reference "#PWR059")
 					(unit 1)
 				)
 				(path "/38b0a34b-2047-47f6-90d7-ccdf77e8e212/b49af01b-ed96-4d9d-b321-2a9fe8fbe5c1/31e52373-a2dc-44cb-afdb-9746210f2a01"
-					(reference "#PWR01")
+					(reference "#PWR031")
 					(unit 1)
 				)
 				(path "/38b0a34b-2047-47f6-90d7-ccdf77e8e212/b49af01b-ed96-4d9d-b321-2a9fe8fbe5c1/37cfab98-42f4-441d-a436-14a61a241678"
-					(reference "#PWR03")
+					(reference "#PWR042")
 					(unit 1)
 				)
 				(path "/38b0a34b-2047-47f6-90d7-ccdf77e8e212/b49af01b-ed96-4d9d-b321-2a9fe8fbe5c1/f6e61053-1e52-4f8f-88d6-a469198d56c4"
-					(reference "#PWR08")
+					(reference "#PWR055")
 					(unit 1)
 				)
@@
 		(dnp no)
 		(fields_autoplaced yes)
-		(property "Reference" "C12"
+		(property "Reference" "C31"
 			(at 80.01 55.8799 0)
 			(effects
@@
 		(instances
 			(project "combat-control"
+				(path "/38b0a34b-2047-47f6-90d7-ccdf77e8e212/5bc2eb48-ba05-4947-b6cc-1fab53bcabc8/31e52373-a2dc-44cb-afdb-9746210f2a01"
+					(reference "C39")
+					(unit 1)
+				)
 				(path "/38b0a34b-2047-47f6-90d7-ccdf77e8e212/5bc2eb48-ba05-4947-b6cc-1fab53bcabc8/37cfab98-42f4-441d-a436-14a61a241678"
-					(reference "C13")
+					(reference "C31")
 					(unit 1)
 				)
 				(path "/38b0a34b-2047-47f6-90d7-ccdf77e8e212/5bc2eb48-ba05-4947-b6cc-1fab53bcabc8/f6e61053-1e52-4f8f-88d6-a469198d56c4"
-					(reference "C14")
+					(reference "C40")
+					(unit 1)
+				)
+				(path "/38b0a34b-2047-47f6-90d7-ccdf77e8e212/b49af01b-ed96-4d9d-b321-2a9fe8fbe5c1/31e52373-a2dc-44cb-afdb-9746210f2a01"
+					(reference "C23")
 					(unit 1)
 				)
 				(path "/38b0a34b-2047-47f6-90d7-ccdf77e8e212/b49af01b-ed96-4d9d-b321-2a9fe8fbe5c1/37cfab98-42f4-441d-a436-14a61a241678"
-					(reference "C12")
+					(reference "C30")
 					(unit 1)
 				)
 				(path "/38b0a34b-2047-47f6-90d7-ccdf77e8e212/b49af01b-ed96-4d9d-b321-2a9fe8fbe5c1/f6e61053-1e52-4f8f-88d6-a469198d56c4"
-					(reference "C11")
+					(reference "C38")
 					(unit 1)
 				)
@@
 		(dnp no)
 		(fields_autoplaced yes)
-		(property "Reference" "#PWR011"
+		(property "Reference" "#PWR058"
 			(at 76.2 95.25 0)
 			(effects
@@
 			(project "combat-control"
 				(path "/38b0a34b-2047-47f6-90d7-ccdf77e8e212/5bc2eb48-ba05-4947-b6cc-1fab53bcabc8/31e52373-a2dc-44cb-afdb-9746210f2a01"
-					(reference "#PWR011")
+					(reference "#PWR058")
 					(unit 1)
 				)
 				(path "/38b0a34b-2047-47f6-90d7-ccdf77e8e212/5bc2eb48-ba05-4947-b6cc-1fab53bcabc8/37cfab98-42f4-441d-a436-14a61a241678"
-					(reference "#PWR06")
+					(reference "#PWR045")
 					(unit 1)
 				)
 				(path "/38b0a34b-2047-47f6-90d7-ccdf77e8e212/5bc2eb48-ba05-4947-b6cc-1fab53bcabc8/f6e61053-1e52-4f8f-88d6-a469198d56c4"
-					(reference "#PWR013")
+					(reference "#PWR060")
 					(unit 1)
 				)
 				(path "/38b0a34b-2047-47f6-90d7-ccdf77e8e212/b49af01b-ed96-4d9d-b321-2a9fe8fbe5c1/31e52373-a2dc-44cb-afdb-9746210f2a01"
-					(reference "#PWR02")
+					(reference "#PWR032")
 					(unit 1)
 				)
 				(path "/38b0a34b-2047-47f6-90d7-ccdf77e8e212/b49af01b-ed96-4d9d-b321-2a9fe8fbe5c1/37cfab98-42f4-441d-a436-14a61a241678"
-					(reference "#PWR04")
+					(reference "#PWR043")
 					(unit 1)
 				)
 				(path "/38b0a34b-2047-47f6-90d7-ccdf77e8e212/b49af01b-ed96-4d9d-b321-2a9fe8fbe5c1/f6e61053-1e52-4f8f-88d6-a469198d56c4"
-					(reference "#PWR09")
+					(reference "#PWR056")
 					(unit 1)
 				)
@@
 		(dnp no)
 		(fields_autoplaced yes)
-		(property "Reference" "R22"
+		(property "Reference" "R24"
 			(at 78.74 81.2799 0)
 			(effects
@@
 			(project "combat-control"
 				(path "/38b0a34b-2047-47f6-90d7-ccdf77e8e212/5bc2eb48-ba05-4947-b6cc-1fab53bcabc8/31e52373-a2dc-44cb-afdb-9746210f2a01"
-					(reference "R22")
+					(reference "R24")
 					(unit 1)
 				)
 				(path "/38b0a34b-2047-47f6-90d7-ccdf77e8e212/5bc2eb48-ba05-4947-b6cc-1fab53bcabc8/37cfab98-42f4-441d-a436-14a61a241678"
-					(reference "R12")
+					(reference "R14")
 					(unit 1)
 				)
 				(path "/38b0a34b-2047-47f6-90d7-ccdf77e8e212/5bc2eb48-ba05-4947-b6cc-1fab53bcabc8/f6e61053-1e52-4f8f-88d6-a469198d56c4"
-					(reference "R26")
+					(reference "R28")
 					(unit 1)
 				)
@@
 				)
 				(path "/38b0a34b-2047-47f6-90d7-ccdf77e8e212/b49af01b-ed96-4d9d-b321-2a9fe8fbe5c1/37cfab98-42f4-441d-a436-14a61a241678"
-					(reference "R8")
+					(reference "R10")
 					(unit 1)
 				)
 				(path "/38b0a34b-2047-47f6-90d7-ccdf77e8e212/b49af01b-ed96-4d9d-b321-2a9fe8fbe5c1/f6e61053-1e52-4f8f-88d6-a469198d56c4"
-					(reference "R18")
+					(reference "R20")
 					(unit 1)
 				)
@@
 		(on_board yes)
 		(dnp no)
-		(property "Reference" "R20"
+		(property "Reference" "R22"
 			(at 49.53 65.786 90)
 			(effects
@@
 			(project "combat-control"
 				(path "/38b0a34b-2047-47f6-90d7-ccdf77e8e212/5bc2eb48-ba05-4947-b6cc-1fab53bcabc8/31e52373-a2dc-44cb-afdb-9746210f2a01"
-					(reference "R20")
+					(reference "R22")
 					(unit 1)
 				)
 				(path "/38b0a34b-2047-47f6-90d7-ccdf77e8e212/5bc2eb48-ba05-4947-b6cc-1fab53bcabc8/37cfab98-42f4-441d-a436-14a61a241678"
-					(reference "R10")
+					(reference "R12")
 					(unit 1)
 				)
 				(path "/38b0a34b-2047-47f6-90d7-ccdf77e8e212/5bc2eb48-ba05-4947-b6cc-1fab53bcabc8/f6e61053-1e52-4f8f-88d6-a469198d56c4"
-					(reference "R24")
+					(reference "R26")
 					(unit 1)
 				)
@@
 				)
 				(path "/38b0a34b-2047-47f6-90d7-ccdf77e8e212/b49af01b-ed96-4d9d-b321-2a9fe8fbe5c1/37cfab98-42f4-441d-a436-14a61a241678"
-					(reference "R6")
+					(reference "R8")
 					(unit 1)
 				)
 				(path "/38b0a34b-2047-47f6-90d7-ccdf77e8e212/b49af01b-ed96-4d9d-b321-2a9fe8fbe5c1/f6e61053-1e52-4f8f-88d6-a469198d56c4"
-					(reference "R15")
+					(reference "R18")
 					(unit 1)
 				)
@@
 		(dnp no)
 		(fields_autoplaced yes)
-		(property "Reference" "R21"
+		(property "Reference" "R23"
 			(at 78.74 68.5799 0)
 			(effects
@@
 			(project "combat-control"
 				(path "/38b0a34b-2047-47f6-90d7-ccdf77e8e212/5bc2eb48-ba05-4947-b6cc-1fab53bcabc8/31e52373-a2dc-44cb-afdb-9746210f2a01"
-					(reference "R21")
+					(reference "R23")
 					(unit 1)
 				)
 				(path "/38b0a34b-2047-47f6-90d7-ccdf77e8e212/5bc2eb48-ba05-4947-b6cc-1fab53bcabc8/37cfab98-42f4-441d-a436-14a61a241678"
-					(reference "R11")
+					(reference "R13")
 					(unit 1)
 				)
 				(path "/38b0a34b-2047-47f6-90d7-ccdf77e8e212/5bc2eb48-ba05-4947-b6cc-1fab53bcabc8/f6e61053-1e52-4f8f-88d6-a469198d56c4"
-					(reference "R25")
+					(reference "R27")
 					(unit 1)
 				)
@@
 				)
 				(path "/38b0a34b-2047-47f6-90d7-ccdf77e8e212/b49af01b-ed96-4d9d-b321-2a9fe8fbe5c1/37cfab98-42f4-441d-a436-14a61a241678"
-					(reference "R7")
+					(reference "R9")
 					(unit 1)
 				)
 				(path "/38b0a34b-2047-47f6-90d7-ccdf77e8e212/b49af01b-ed96-4d9d-b321-2a9fe8fbe5c1/f6e61053-1e52-4f8f-88d6-a469198d56c4"
-					(reference "R17")
+					(reference "R19")
 					(unit 1)
 				)
@@
 		(on_board yes)
 		(dnp no)
-		(property "Reference" "R1"
+		(property "Reference" "R21"
 			(at 49.53 50.546 90)
 			(effects
@@
 			(project "combat-control"
 				(path "/38b0a34b-2047-47f6-90d7-ccdf77e8e212/5bc2eb48-ba05-4947-b6cc-1fab53bcabc8/31e52373-a2dc-44cb-afdb-9746210f2a01"
-					(reference "R19")
+					(reference "R21")
 					(unit 1)
 				)
 				(path "/38b0a34b-2047-47f6-90d7-ccdf77e8e212/5bc2eb48-ba05-4947-b6cc-1fab53bcabc8/37cfab98-42f4-441d-a436-14a61a241678"
-					(reference "R9")
+					(reference "R11")
 					(unit 1)
 				)
 				(path "/38b0a34b-2047-47f6-90d7-ccdf77e8e212/5bc2eb48-ba05-4947-b6cc-1fab53bcabc8/f6e61053-1e52-4f8f-88d6-a469198d56c4"
-					(reference "R23")
+					(reference "R25")
 					(unit 1)
 				)
@@
 				)
 				(path "/38b0a34b-2047-47f6-90d7-ccdf77e8e212/b49af01b-ed96-4d9d-b321-2a9fe8fbe5c1/37cfab98-42f4-441d-a436-14a61a241678"
-					(reference "R5")
+					(reference "R7")
 					(unit 1)
 				)
 				(path "/38b0a34b-2047-47f6-90d7-ccdf77e8e212/b49af01b-ed96-4d9d-b321-2a9fe8fbe5c1/f6e61053-1e52-4f8f-88d6-a469198d56c4"
-					(reference "R14")
-					(unit 1)
-				)
+					(reference "R17")
+					(unit 1)
+				)

Commit message: Save layout
Parts:
- renumbered C31 to C39
Changed lines of the file:
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@@
 		(dnp no)
 		(fields_autoplaced yes)
-		(property "Reference" "C31"
+		(property "Reference" "C39"
 			(at 80.01 55.8799 0)
 			(effects
