File: pcb/small-motor.kicad_sch (KiCad schematic)
At the start: 1 part

Commit message: Save progress
Parts:
- removed R16: 2m, Resistor_SMD:R_1206_3216Metric, symbol Device:R
- added C15: C, symbol Device:C
- added C17: 10u, Capacitor_SMD:C_0603_1608Metric, symbol Device:C
- added C18, C22: 100n, Capacitor_SMD:C_0402_1005Metric, symbol Device:C
- added C20: 10u, Capacitor_SMD:C_0805_2012Metric, symbol Device:C
- added C21: 470n, Capacitor_SMD:C_0603_1608Metric, symbol Device:C
- added J1, J3, J5: Conn_01x01_Pin, symbol Connector:Conn_01x01_Pin
- added R13: 2m, Resistor_SMD:R_1206_3216Metric, symbol Device:R
- added R33: R, symbol Device:R
- added U2: DRV8328B, Package_DFN_QFN:QFN-28-1EP_4x4mm_P0.4mm_EP2.6x2.6mm, symbol User_Symbols:DRV8328B
Connections:
- net GND: now also C15.2, C17.2, C18.2, C20.2, C22.2, R13.2, U2.27 (DT), U2.28 (GND), U2.29 (PAD)
- net ILIM: now also C15.1, R33.1
- net INA: now also U2.20 (INHA)
- net INB: now also U2.19 (INHB)
- net INC: now also U2.18 (INHC)
- new net: C21.1, U2.2 (CPL)
- new net: C21.2, U2.3 (CPH)
- new net +3V3: U2.21 (INLC), U2.22 (INLB), U2.23 (INLA), U2.25 (~{SLP})
- new net BSTA: U2.5 (BSTA)
- new net BSTB: U2.9 (BSTB)
- new net BSTC: U2.13 (BSTC)
- new net DL: R33.2, U2.26 (DLVL)
- new net GVDD: C17.1, C18.1, U2.4 (GVDD)
- new net HIA: U2.7 (GHA)
- new net HIB: U2.11 (GHB)
- new net HIC: U2.15 (GHC)
- new net LOA: U2.8 (GLA)
- new net LOB: U2.12 (GLB)
- new net LOC: U2.16 (GLC)
- new net LOW: R13.1, U2.17 (LSS)
- new net OUTA: J1.1 (Pin_1), U2.6 (SHA)
- new net OUTB: J3.1 (Pin_1), U2.10 (SHB)
- new net OUTC: J5.1 (Pin_1), U2.14 (SHC)
- new net VDD: C20.1, C22.1, U2.1 (PVDD)
- no-connect marks 0 -> 1
Other:
- sheet SmallBridgeA ports: added BST, GH, GL, LOW, OUT, SNS; removed none
- sheet SmallBridgeB ports: added BST, GH, GL, LOW, OUT, SNS; removed none
- sheet SmallBridgeC ports: added BST, GH, GL, LOW, OUT, SNS; removed none
- note removed: "DRV8328B"

Commit message: Save test layout
Parts:
- removed J3, J5: Conn_01x01_Pin, symbol Connector:Conn_01x01_Pin
- added J4, J7: Conn_01x01_Pin, User_Footprints:Pad-P1.5, symbol Connector:Conn_01x01_Pin
- C34: renamed from C15; footprint (none) -> Capacitor_SMD:C_0402_1005Metric
- J6: renamed from J1; footprint (none) -> User_Footprints:Pad-P1.5; now not fitted; now left out of the parts list
- R15: renamed from R33; footprint (none) -> Resistor_SMD:R_0402_1005Metric
- renumbered C17 to C32, C18 to C33, C20 to C35, C21 to C36, C22 to C37, R13 to R16, U2 to U4
Connections:
- net OUTB: now also J4.1 (Pin_1)
- net OUTC: now also J7.1 (Pin_1)

Commit message: Save layout
Parts:
- renumbered J4 to J5, J7 to J8
Changed lines of the file:
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@@
 		(on_board yes)
 		(dnp yes)
-		(property "Reference" "J4"
+		(property "Reference" "J5"
 			(at 156.972 55.88 0)
 			(effects
@@
 		(on_board yes)
 		(dnp yes)
-		(property "Reference" "J7"
+		(property "Reference" "J8"
 			(at 156.972 76.2 0)
 			(effects
