File: pcb/combat-control.kicad_pcb (KiCad board)
At the start: 4 copper layers, 0 parts

Commit message: Save test layout
Parts:
- added AE1: Antenna_Shield, Connector_Coaxial:U.FL_Molex_MCRF_73412-0110_Vertical, F.Cu at (81.7, 54.4)
- added C1: 4u7, Capacitor_SMD:C_0402_1005Metric, F.Cu at (92.2, 59.7)
- added C10: C, Resistor_SMD:R_0402_1005Metric, F.Cu at (89.4, 59.7)
- added C11: 1u, Capacitor_SMD:C_0402_1005Metric, F.Cu at (95.1, 61.6)
- added C12: 10n, Capacitor_SMD:C_0402_1005Metric, F.Cu at (95.1, 63.6)
- added C13: C, Resistor_SMD:R_0402_1005Metric, F.Cu at (89.4, 61.7)
- added C14: 100n, Capacitor_SMD:C_0402_1005Metric, F.Cu at (95.1, 65.6)
- added C15: 100n, Capacitor_SMD:C_0402_1005Metric, F.Cu at (98.0, 59.7)
- added C16: 100n, Capacitor_SMD:C_0402_1005Metric, F.Cu at (98.0, 61.6)
- added C17: 100n, Capacitor_SMD:C_0402_1005Metric, F.Cu at (98.0, 63.6)
- added C18: 1u, Capacitor_SMD:C_0402_1005Metric, F.Cu at (98.0, 65.6)
- added C19: C, Capacitor_SMD:C_0402_1005Metric, F.Cu at (100.9, 59.7)
- added C2: 100n, Capacitor_SMD:C_0402_1005Metric, F.Cu at (92.2, 61.6)
- added C20: 100n, Capacitor_SMD:C_0402_1005Metric, F.Cu at (100.9, 61.6)
- added C21: C, Capacitor_SMD:C_0402_1005Metric, F.Cu at (100.9, 63.6)
- added C22: C, Capacitor_SMD:C_0402_1005Metric, F.Cu at (100.9, 65.6)
- added C23: 1u, Capacitor_SMD:C_0402_1005Metric, B.Cu at (85.3, 58.6)
- added C24: 10u, Capacitor_SMD:C_0603_1608Metric, B.Cu at (87.7, 56.9)
- added C25: 100n, Capacitor_SMD:C_0402_1005Metric, B.Cu at (87.5, 50.3)
- added C26: C, Capacitor_SMD:C_0402_1005Metric, B.Cu at (87.5, 52.3)
- added C27: 10u, Capacitor_SMD:C_0805_2012Metric, B.Cu at (91.1, 58.0)
- added C28: 470n, Capacitor_SMD:C_0603_1608Metric, B.Cu at (87.7, 59.4)
- added C29: 100n, Capacitor_SMD:C_0402_1005Metric, B.Cu at (87.5, 54.2)
- added C3: 100n, Capacitor_SMD:C_0402_1005Metric, F.Cu at (92.2, 63.6)
- added C30: 1u, Capacitor_SMD:C_0402_1005Metric, B.Cu at (81.2, 50.1)
- added C31: 1u, Capacitor_SMD:C_0402_1005Metric, B.Cu at (81.6, 63.1)
- added C32: 10u, Capacitor_SMD:C_0603_1608Metric, B.Cu at (88.6, 68.8)
- added C33: 100n, Capacitor_SMD:C_0402_1005Metric, B.Cu at (88.5, 62.2)
- added C34: C, Capacitor_SMD:C_0402_1005Metric, B.Cu at (88.5, 64.2)
- added C35: 10u, Capacitor_SMD:C_0805_2012Metric, B.Cu at (91.9, 69.8)
- added C36: 470n, Capacitor_SMD:C_0603_1608Metric, B.Cu at (88.6, 71.3)
- added C37: 100n, Capacitor_SMD:C_0402_1005Metric, B.Cu at (88.5, 66.1)
- added C38: 1u, Capacitor_SMD:C_0402_1005Metric, B.Cu at (83.2, 59.0)
- added C39: 1u, Capacitor_SMD:C_0402_1005Metric, B.Cu at (85.7, 72.0)
- added C4: 2m2, User_Footprints:C_D10xL16_Horizontal, B.Cu at (106.4, 68.4)
- added C40: 1u, Capacitor_SMD:C_0402_1005Metric, B.Cu at (83.7, 72.0)
- added C41: 22u, Capacitor_SMD:C_0805_2012Metric, F.Cu at (116.8, 32.6)
- added C42: 100n, Capacitor_SMD:C_0402_1005Metric, F.Cu at (121.8, 36.4)
- added C43: 10u, Capacitor_SMD:C_0805_2012Metric, F.Cu at (116.8, 35.6)
- added C44: 10u, Capacitor_SMD:C_0805_2012Metric, F.Cu at (116.8, 38.6)
- added C45: 470n, Capacitor_SMD:C_0603_1608Metric, F.Cu at (116.5, 41.4)
- added C46: 100n, Capacitor_SMD:C_0402_1005Metric, F.Cu at (121.8, 38.4)
- added C47: 100n, Capacitor_SMD:C_0402_1005Metric, F.Cu at (121.8, 40.3)
- added C48: 10u, Capacitor_SMD:C_0603_1608Metric, F.Cu at (146.4, 60.9)
- added C49: 10u, Capacitor_SMD:C_0603_1608Metric, F.Cu at (145.0, 79.8)
- added C50: 10u, Capacitor_SMD:C_0603_1608Metric, F.Cu at (146.4, 47.3)
- added C6: 2m2, User_Footprints:C_D10xL16_Horizontal, B.Cu at (106.2, 58.4)
- added C8: 1u, Capacitor_SMD:C_0402_1005Metric, F.Cu at (92.2, 65.6)
- added C9: 10u, Capacitor_SMD:C_0402_1005Metric, F.Cu at (95.1, 59.7)
- added J1: Conn_01x01_Pin, MountingHole:MountingHole_3.2mm_M3_Pad_Via, F.Cu at (112.2, 71.2)
- added J2: Conn_01x01_Pin, MountingHole:MountingHole_3.2mm_M3_Pad_Via, F.Cu at (111.6, 49.6)
- added J2: Conn_01x01_Pin, MountingHole:MountingHole_3.2mm_M3_Pad_Via, F.Cu at (132.6, 71.1)
- added J2: Conn_01x01_Pin, MountingHole:MountingHole_3.2mm_M3_Pad_Via, F.Cu at (132.4, 60.4)
- added J2: Conn_01x01_Pin, MountingHole:MountingHole_3.2mm_M3_Pad_Via, F.Cu at (132.8, 49.3)
- added J3: Conn_01x01_Pin, User_Footprints:Pad-P1.5, F.Cu at (96.4, 48.0)
- added J4: Conn_01x01_Pin, User_Footprints:Pad-P1.5, F.Cu at (100.0, 48.0)
- added J5: Conn_01x01_Pin, User_Footprints:Pad-P1.5, F.Cu at (100.0, 73.2)
- added J6: Conn_01x01_Pin, User_Footprints:Pad-P1.5, F.Cu at (103.2, 73.0)
- added J7: Conn_01x01_Pin, User_Footprints:Pad-P1.5, F.Cu at (103.4, 48.0)
- added J8: Conn_01x01_Pin, User_Footprints:Pad-P1.5, F.Cu at (96.4, 73.2)
- added L1: L, Inductor_SMD:L_0402_1005Metric, F.Cu at (89.4, 63.6)
- added L2: 2nH, Inductor_SMD:L_0402_1005Metric, F.Cu at (89.4, 65.6)
- added L3: L, Inductor_SMD:L_0402_1005Metric, F.Cu at (89.4, 67.6)
- added L4: L, Inductor_SMD:L_0402_1005Metric, F.Cu at (89.4, 69.6)
- added Q1: AON7544, User_Footprints:DFN3x3A_8L_EP1_P, B.Cu at (96.7, 51.7)
- added Q10: AON7544, User_Footprints:DFN3x3A_8L_EP1_P, F.Cu at (103.0, 69.6)
- added Q11: AON7544, User_Footprints:DFN3x3A_8L_EP1_P, B.Cu at (96.7, 69.6)
- added Q12: AON7544, User_Footprints:DFN3x3A_8L_EP1_P, F.Cu at (96.6, 69.6)
- added Q2: AON7544, User_Footprints:DFN3x3A_8L_EP1_P, F.Cu at (96.7, 51.8)
- added Q3: AON7544, User_Footprints:DFN3x3A_8L_EP1_P, B.Cu at (99.9, 51.7)
- added Q4: AON7544, User_Footprints:DFN3x3A_8L_EP1_P, F.Cu at (100.0, 51.8)
- added Q5: AON7544, User_Footprints:DFN3x3A_8L_EP1_P, B.Cu at (99.9, 69.6)
- added Q6: AON7544, User_Footprints:DFN3x3A_8L_EP1_P, F.Cu at (99.8, 69.6)
- added Q7: AON7544, User_Footprints:DFN3x3A_8L_EP1_P, B.Cu at (103.1, 51.7)
- added Q8: AON7544, User_Footprints:DFN3x3A_8L_EP1_P, F.Cu at (103.2, 51.8)
- added Q9: AON7544, User_Footprints:DFN3x3A_8L_EP1_P, B.Cu at (103.1, 69.6)
- added R1: 22R, Resistor_SMD:R_0402_1005Metric, B.Cu at (85.2, 50.4)
- added R10: 1k, Resistor_SMD:R_0402_1005Metric, B.Cu at (81.1, 59.0)
- added R11: 22R, Resistor_SMD:R_0402_1005Metric, B.Cu at (81.5, 66.1)
- added R12: 22R, Resistor_SMD:R_0402_1005Metric, B.Cu at (81.5, 68.1)
- added R13: 4k7, Resistor_SMD:R_0402_1005Metric, B.Cu at (81.5, 70.1)
- added R14: 1k, Resistor_SMD:R_0402_1005Metric, B.Cu at (81.5, 72.1)
- added R15: R, Resistor_SMD:R_0402_1005Metric, B.Cu at (89.1, 73.5)
- added R16: 2m, Resistor_SMD:R_1206_3216Metric, F.Cu at (103.0, 65.4)
- added R17: 22R, Resistor_SMD:R_0402_1005Metric, B.Cu at (83.1, 50.4)
- added R18: 22R, Resistor_SMD:R_0402_1005Metric, B.Cu at (83.1, 52.3)
- added R19: 4k7, Resistor_SMD:R_0402_1005Metric, B.Cu at (83.1, 54.3)
- added R2: 22R, Resistor_SMD:R_0402_1005Metric, B.Cu at (85.2, 52.4)
- added R20: 1k, Resistor_SMD:R_0402_1005Metric, B.Cu at (83.1, 56.3)
- added R21: 22R, Resistor_SMD:R_0402_1005Metric, B.Cu at (85.6, 63.8)
- added R22: 22R, Resistor_SMD:R_0402_1005Metric, B.Cu at (85.6, 65.7)
- added R23: 4k7, Resistor_SMD:R_0402_1005Metric, B.Cu at (85.6, 67.7)
- added R24: 1k, Resistor_SMD:R_0402_1005Metric, B.Cu at (85.6, 69.7)
- added R25: 22R, Resistor_SMD:R_0402_1005Metric, B.Cu at (83.6, 63.4)
- added R26: 22R, Resistor_SMD:R_0402_1005Metric, B.Cu at (83.6, 65.3)
- added R27: 4k7, Resistor_SMD:R_0402_1005Metric, B.Cu at (83.6, 67.3)
- added R28: 1k, Resistor_SMD:R_0402_1005Metric, B.Cu at (83.6, 69.3)
- added R29: 10k, Resistor_SMD:R_0402_1005Metric, F.Cu at (116.0, 43.6)
- added R3: 4k7, Resistor_SMD:R_0402_1005Metric, B.Cu at (85.2, 54.4)
- added R30: 22R, Resistor_SMD:R_0603_1608Metric, F.Cu at (146.4, 58.4)
- added R31: 22R, Resistor_SMD:R_0603_1608Metric, F.Cu at (146.4, 55.9)
- added R32: 15k, Resistor_SMD:R_0402_1005Metric, F.Cu at (146.9, 53.6)
- added R33: 2k, Resistor_SMD:R_0402_1005Metric, F.Cu at (146.9, 51.6)
- added R34: 22R, Resistor_SMD:R_0603_1608Metric, F.Cu at (145.0, 77.3)
- added R35: 22R, Resistor_SMD:R_0603_1608Metric, F.Cu at (145.0, 74.8)
- added R36: 15k, Resistor_SMD:R_0402_1005Metric, F.Cu at (145.5, 72.5)
- added R37: 2k, Resistor_SMD:R_0402_1005Metric, F.Cu at (145.5, 70.6)
- added R38: 22R, Resistor_SMD:R_0603_1608Metric, F.Cu at (146.4, 44.8)
- added R39: 22R, Resistor_SMD:R_0603_1608Metric, F.Cu at (146.4, 42.2)
- added R4: 1k, Resistor_SMD:R_0402_1005Metric, B.Cu at (85.2, 56.4)
- added R40: 15k, Resistor_SMD:R_0402_1005Metric, F.Cu at (146.9, 40.0)
- added R41: 2k, Resistor_SMD:R_0402_1005Metric, F.Cu at (146.9, 38.0)
- added R5: R, Resistor_SMD:R_0402_1005Metric, B.Cu at (85.2, 60.0)
- added R6: 2m, Resistor_SMD:R_1206_3216Metric, F.Cu at (103.2, 56.6)
- added R7: 22R, Resistor_SMD:R_0402_1005Metric, B.Cu at (81.1, 53.0)
- added R8: 22R, Resistor_SMD:R_0402_1005Metric, B.Cu at (81.1, 55.0)
- added R9: 4k7, Resistor_SMD:R_0402_1005Metric, B.Cu at (81.1, 57.0)
- added U1: ICM-42688-P, Package_LGA:LGA-14_3x2.5mm_P0.5mm_LayoutBorder3x4y, F.Cu at (85.2, 68.6)
- added U10: TPHR8504PL, Package_DFN_QFN:PQFN-8-EP_6x5mm_P1.27mm_Generic, F.Cu at (125.1, 67.3)
- added U11: TPHR8504PL, Package_DFN_QFN:PQFN-8-EP_6x5mm_P1.27mm_Generic, B.Cu at (125.4, 53.2)
- added U12: TPHR8504PL, Package_DFN_QFN:PQFN-8-EP_6x5mm_P1.27mm_Generic, F.Cu at (125.1, 53.0)
- added U2: ESP32-S3, Package_DFN_QFN:QFN-56-1EP_7x7mm_P0.4mm_EP4x4mm, F.Cu at (82.7, 61.7)
- added U3: DRV8328B, Package_DFN_QFN:QFN-28-1EP_4x4mm_P0.4mm_EP2.6x2.6mm, B.Cu at (91.5, 52.6)
- added U4: DRV8328B, Package_DFN_QFN:QFN-28-1EP_4x4mm_P0.4mm_EP2.6x2.6mm, B.Cu at (93.0, 64.3)
- added U5: DRV8328B, Package_DFN_QFN:QFN-28-1EP_4x4mm_P0.4mm_EP2.6x2.6mm, F.Cu at (112.0, 64.4)
- added U6: ACS781xLRTR-100B, Sensor_Current:Allegro_PSOF-7_4.8x6.4mm_P1.60mm, F.Cu at (111.4, 57.2)
- added U7: TPHR8504PL, Package_DFN_QFN:PQFN-8-EP_6x5mm_P1.27mm_Generic, B.Cu at (125.4, 60.5)
- added U8: TPHR8504PL, Package_DFN_QFN:PQFN-8-EP_6x5mm_P1.27mm_Generic, F.Cu at (125.1, 60.4)
- added U9: TPHR8504PL, Package_DFN_QFN:PQFN-8-EP_6x5mm_P1.27mm_Generic, B.Cu at (125.2, 67.3)
- added Y1: 40MHz, Crystal:Crystal_SMD_2520-4Pin_2.5x2.0mm, F.Cu at (81.2, 68.5)
Routing:
- net Net-(U9-G): track 0.00 -> 1.10 mm, vias 0 -> 1
Other:
- board outline added: 59 x 30.2 mm

Commit message: Save layout
Parts:
- removed C6: 2m2, User_Footprints:C_D10xL16_Horizontal
- removed the J2 at (111.6, 49.6)
- removed the J2 at (132.6, 71.1)
- removed the J2 at (132.4, 60.4)
- removed the J2 at (132.8, 49.3)
- added C5: 2m2, User_Footprints:C_D10xL16_Horizontal, B.Cu at (119.5, 58.2)
- added J10: Conn_01x01_Pin, MountingHole:MountingHole_3.2mm_M3_Pad_Via, F.Cu at (136.0, 63.8)
- added J11: Conn_01x01_Pin, MountingHole:MountingHole_3.2mm_M3_Pad_Via, F.Cu at (135.9, 56.2)
- added J2: Conn_01x01_Pin, MountingHole:MountingHole_3.2mm_M3_Pad_Via, F.Cu at (110.1, 71.5)
- added J9: Conn_01x01_Pin, MountingHole:MountingHole_3.2mm_M3_Pad_Via, F.Cu at (136.0, 71.4)
- C23, C24, C25, C26, C27, C28, C29, C30, C31, C32, C33, C34, C35, C36, C37, C38, C39, C40, R10, R12, R13, R14, R15, R18, R19, R2, R20, R22, R23, R24, R26, R27, R28, R3, R4, R5, R8, R9: moved to F.Cu
- C41, C42, C43, C44, C46, R30, R34, R38: moved to B.Cu
- moved C19 41.6 mm to (59.5, 64.5), turned to 90 degrees
- moved C49 40.9 mm to (114.9, 52.1), turned to 90 degrees
- moved C21 39.3 mm to (61.5, 64.3), turned to 90 degrees
- moved C22 37.4 mm to (63.5, 64.3), turned to 90 degrees
- moved C20 36.6 mm to (64.7, 55.9), turned to 90 degrees
- moved C48 32.4 mm to (114.5, 55.4), turned to 90 degrees
- moved C50 32.1 mm to (114.3, 48.8), turned to 90 degrees
- moved C15 31.3 mm to (67.2, 65.0), turned to 90 degrees
- moved C12 31.2 mm to (64.1, 60.5), turned to 90 degrees
- moved L1 30.3 mm to (59.6, 58.0), turned to 90 degrees
- moved C10 28.9 mm to (60.7, 55.7), turned to 90 degrees
- moved C9 28.8 mm to (67.4, 67.3), turned to 90 degrees
- moved C17 28.0 mm to (72.5, 52.1), turned to 90 degrees
- moved C18 28.0 mm to (73.5, 52.1), turned to 90 degrees
- moved L3 27.7 mm to (61.7, 67.5), turned to 90 degrees
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Connections:
- C4 pad 2: GND -> /LargeMotor/LOW
- U2 pad 5: unconnected-(U2-GPIO0-Pad5) -> /IFIG
- U2 pad 51: unconnected-(U2-GPIO45-Pad51) -> /IFIG
- U6 pad 5: /LargeMotor/LOW -> GND
- U6 pad 6: GND -> /LargeMotor/LOW
Routing:
- net Net-(U9-G): track 1.10 -> 0.00 mm, vias 1 -> 0
Other:
- board size 59 x 30.2 mm -> 61.6 x 22.5 mm

Commit message: Save layout
Parts:
- moved R31 0.39 mm to (126.6, 73.8)
- moved U8 0.25 mm to (128.7, 70.2)
- moved R35 0.19 mm to (126.6, 66.6)
- moved U10 0.17 mm to (128.6, 62.9)
